Commit message: feat: fix typo, fix reverse joints, fix joint rotation on urdf and refactor rviz_server_node

File: urdf/robot.urdf (robot description, URDF)
Before this commit: robot arpis, 35 links, 34 joints
Joints:
- joint head: origin xyz=0 .0 .12 rpy=0 0 0 -> xyz=0 .0 .03 rpy=0 0 0
- joint head_tilt: origin xyz=0 .0 .05 rpy=0 0 0 -> xyz=0 .0 .05 rpy=0.5 0 0
- joint left_hip_yaw: origin xyz=-0.15 0 -.45 rpy=0 0 0 -> xyz=-0.15 0 -.45 rpy=0 0.03 0
- joint right_hip_yaw: origin xyz=0.15 0 -.45 rpy=0 0 0 -> xyz=0.15 0 -.45 rpy=0 .05 0
- joint right_shoulder_roll: origin xyz=0 .0 -0.15 rpy=0 -0.35 0 -> xyz=0 .0 -0.15 rpy=0 -0.7 0
